File: Operant/Nosepoke/KiCadFiles/NosepokeV1.0.kicad_pcb (KiCad board)
At the start: 2 copper layers, 28 x 45 mm, 29 parts, among them J1 SSW-102-02-T-S-RA, J2 SSW-102-02-T-S-RA, J3 5V power in, J4 SPI in, J5 I2C in, J6 SPI out, J7 I2C out, J8 Conn_01x03, Q1 BSS138, Q2 BSS138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

Commit message: CAD drawings added
CAD drawings for operant unit added
Other:
- net class Default removed
- net class POWER removed
